File: disco_fish.kicad_pcb (KiCad board)
At the start: 2 copper layers, 60 x 100 mm, 55 parts, among them J1 EBBA-04-C-SS-BU, J10 Conn_02x03, J2 EBBA-04-C-SS-BU, J3 EBBA-04-C-SS-BU, J4 EBBA-04-C-SS-BU, J5 EBBA-04-C-SS-BU, J6 EBBA-04-C-SS-BU, J7 EBBA-04-C-SS-BU, J8 EBBA-04-C-SS-BU, J9 Barrel_Jack_Mounting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

Commit message: finalized design
Parts:
- J9: value Barrel_Jack_Mounting -> EBBA-04-C-SS-BU; footprint personal:barrel_jack_mounting -> personal:EBBA-04-C-SS-BU
- moved J9 14.2 mm to (172.5, 46.0), turned to 180 degrees
Routing:
- net GND: track 97.1 -> 81.8 mm, vias 48 -> 40
Other:
- board text added: "12V"
Changed lines of the file:
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@@
   (general
     (thickness 1.6)
-    (drawings 64)
-    (tracks 364)
+    (drawings 68)
+    (tracks 344)
     (zones 0)
     (modules 55)
@@
       (outputformat 1)
       (mirror false)
-      (drillshape 1)
+      (drillshape 0)
       (scaleselection 1)
-      (outputdirectory ""))
+      (outputdirectory "disco_fish_gerber/"))
   )
   (net 0 "")
@@
       (xy 10.64054 17.646415) (xy 10.723619 17.653) (xy 10.937147 17.625795)) (layer B.SilkS) (width 0.01))
   )
-  (module personal:barrel_jack_mounting (layer F.Cu)
-    (at 160.655 53.848 270)
-    (fp_text reference J9 (at -10.16 -5.588 180) (layer F.SilkS)
-      (effects (font (size 0.762 0.762) (thickness 0.127)))
-    )
-    (fp_text value Barrel_Jack_Mounting (at -3.556 6.096 90) (layer F.Fab)
-      (effects (font (size 0.762 0.762) (thickness 0.127)))
-    )
-    (fp_text user "pcb edge" (at -10.668 0.254 180) (layer Dwgs.User)
-      (effects (font (size 1 1) (thickness 0.15)))
-    )
-    (fp_line (start -11.5 5.2) (end -11.5 -4.3) (layer F.SilkS) (width 0.12))
-    (fp_line (start 3 5.2) (end 3 -4.3) (layer F.SilkS) (width 0.12))
-    (fp_line (start 3 -4.3) (end -11.5 -4.3) (layer F.SilkS) (width 0.12))
-    (fp_line (start 3 5.2) (end -11.5 5.2) (layer F.SilkS) (width 0.12))
-    (pad 1 thru_hole rect (at 3 0 90) (size 1.5 3.5) (drill oval 1 3) (layers *.Cu *.Mask)
-      (net 2 /12V))
-    (pad 3 thru_hole rect (at 0 4.7) (size 1.5 3.5) (drill oval 1 3) (layers *.Cu *.Mask)
-      (net 1 GND))
-    (pad 2 thru_hole rect (at -3 0 270) (size 1.5 3.5) (drill oval 1 3) (layers *.Cu *.Mask)
-      (net 1 GND))
-  )
   (module Housings_DIP:DIP-28_W7.62mm (layer F.Cu)
     (at 161.163 74.676)
@@
     (pad 1 smd rect (at -0.85 -1.1) (size 1.2 1.4) (layers F.Cu F.Paste F.Mask)
       (net 4 "Net-(C3-Pad1)"))
+  )
+  (module personal:EBBA-04-C-SS-BU (layer F.Cu)
+    (at 172.513 45.974 180)
+    (fp_text reference J9 (at -3.763 -3.556) (layer F.SilkS)
+      (effects (font (size 1 1) (thickness 0.15)))
+    )
+    (fp_text value EBBA-04-C-SS-BU (at 7.874 -3.302) (layer F.Fab) hide
+      (effects (font (size 1 1) (thickness 0.15)))
+    )
+    (fp_line (start -2.75 -4.2) (end 17.75 -4.2) (layer F.SilkS) (width 0.12))
+    (fp_line (start -2.75 3.4) (end 17.75 3.4) (layer F.SilkS) (width 0.12))
+    (fp_line (start -2.75 3.4) (end -2.75 -4.2) (layer F.SilkS) (width 0.12))
+    (fp_line (start 17.75 -4.2) (end 17.75 3.4) (layer F.SilkS) (width 0.12))
+    (fp_text user "pcb edge" (at 7.493 2.794) (layer Dwgs.User)
+      (effects (font (size 1 1) (thickness 0.15)))
+    )
+    (pad 1 thru_hole circle (at 0 0) (size 1.8 1.8) (drill 1.2) (layers *.Cu *.Mask)
+      (net 2 /12V))
+    (pad 2 thru_hole circle (at 5 0) (size 1.8 1.8) (drill 1.2) (layers *.Cu *.Mask)
+      (net 1 GND))
+    (pad 3 thru_hole circle (at 10 0) (size 1.8 1.8) (drill 1.2) (layers *.Cu *.Mask)
+      (net 1 GND))
+    (pad 4 thru_hole circle (at 15 0) (size 1.8 1.8) (drill 1.2) (layers *.Cu *.Mask)
+      (net 2 /12V))
+  )
+  (gr_text 12V (at 172.974 53.086 90) (layer F.SilkS)
+    (effects (font (size 1.778 1.778) (thickness 0.3048)))
+  )
+  (gr_text 12V (at 157.734 53.086 90) (layer F.SilkS)
+    (effects (font (size 1.778 1.778) (thickness 0.3048)))
+  )
+  (gr_text GND (at 167.64 53.086 90) (layer F.SilkS)
+    (effects (font (size 1.778 1.778) (thickness 0.3048)))
+  )
+  (gr_text GND (at 162.56 53.086 90) (layer F.SilkS)
+    (effects (font (size 1.778 1.778) (thickness 0.3048)))
   )
   (gr_text "DISCO FISH" (at 147.828 141.224) (layer F.SilkS)
@@
   (segment (start 184.166 134.604) (end 184.15 134.62) (width 1.016) (layer F.Cu) (net 1))
   (segment (start 184.166 133.492) (end 184.166 134.604) (width 1.016) (layer F.Cu) (net 1))
-  (via (at 154.686 53.848) (size 0.8128) (drill 0.4064) (layers F.Cu B.Cu) (net 1))
-  (segment (start 155.955 53.848) (end 154.686 53.848) (width 1.016) (layer F.Cu) (net 1))
-  (via (at 160.655 52.07) (size 0.8128) (drill 0.4064) (layers F.Cu B.Cu) (net 1))
-  (segment (start 160.655 50.848) (end 160.655 52.07) (width 1.016) (layer F.Cu) (net 1))
   (segment (start 158.777 95.801) (end 158.877 95.901) (width 0.254) (layer F.Cu) (net 1))
   (segment (start 156.933 95.801) (end 158.777 95.801) (width 0.254) (layer F.Cu) (net 1))
@@
   (segment (start 168.807 59.46) (end 168.783 59.436) (width 0.508) (layer F.Cu) (net 1))
   (segment (start 168.807 63.372) (end 168.807 59.46) (width 0.508) (layer F.Cu) (net 1))
-  (via (at 157.353 53.848) (size 0.8128) (drill 0.4064) (layers F.Cu B.Cu) (net 1))
-  (segment (start 155.955 53.848) (end 157.353 53.848) (width 1.016) (layer F.Cu) (net 1))
-  (via (at 160.655 49.53) (size 0.8128) (drill 0.4064) (layers F.Cu B.Cu) (net 1))
-  (segment (start 160.655 50.848) (end 160.655 49.53) (width 1.016) (layer F.Cu) (net 1))
-  (segment (start 155.955 51.436) (end 155.956 51.435) (width 1.016) (layer F.Cu) (net 1))
-  (via (at 155.956 51.435) (size 0.8128) (drill 0.4064) (layers F.Cu B.Cu) (net 1))
-  (segment (start 155.955 53.848) (end 155.955 51.436) (width 1.016) (layer F.Cu) (net 1))
-  (via (at 155.956 56.261) (size 0.8128) (drill 0.4064) (layers F.Cu B.Cu) (net 1))
-  (segment (start 155.955 56.26) (end 155.956 56.261) (width 1.016) (layer F.Cu) (net 1))
-  (segment (start 155.955 53.848) (end 155.955 56.26) (width 1.016) (layer F.Cu) (net 1))
-  (via (at 163.195 50.8) (size 0.8128) (drill 0.4064) (layers F.Cu B.Cu) (net 1))
-  (segment (start 163.147 50.848) (end 163.195 50.8) (width 1.016) (layer F.Cu) (net 1))
-  (segment (start 160.655 50.848) (end 163.147 50.848) (width 1.016) (layer F.Cu) (net 1))
-  (via (at 157.988 50.927) (size 0.8128) (drill 0.4064) (layers F.Cu B.Cu) (net 1))
-  (segment (start 158.067 50.848) (end 157.988 50.927) (width 1.016) (layer F.Cu) (net 1))
-  (segment (start 160.655 50.848) (end 158.067 50.848) (width 1.016) (layer F.Cu) (net 1))
   (via (at 172.593 59.69) (size 0.8128) (drill 0.4064) (layers F.Cu B.Cu) (net 1))
   (segment (start 168.911 63.372) (end 172.593 59.69) (width 0.508) (layer F.Cu) (net 1))
@@
   (segment (start 171.45 105.156) (end 171.704 104.902) (width 0.508) (layer F.Cu) (net 43))
   (segment (start 168.783 105.156) (end 171.45 105.156) (width 0.254) (layer F.Cu) (net 43))
+  (zone (net 2) (net_name /12V) (layer F.Cu) (hatch edge 0.508)
+    (connect_pads yes (clearance 0.3048))
+    (min_thickness 0.381)
+    (fill yes (arc_segments 32) (thermal_gap 0.508) (thermal_bridge_width 0.508))
+    (polygon
+      (pts
+        (xy 198.247 145.161) (xy 186.817 145.161) (xy 186.817 63.373) (xy 143.383 63.373) (xy 143.383 145.161)
+        (xy 134.366 145.161) (xy 134.366 39.624) (xy 198.247 39.624)
+      )
+    )
+  )
   (zone (net 1) (net_name GND) (layer B.Cu) (hatch edge 0.508)
     (priority 2)
@@
       )
     )
-  )
-  (zone (net 2) (net_name /12V) (layer F.Cu) (hatch edge 0.508)
-    (connect_pads yes (clearance 0.3048))
-    (min_thickness 0.381)
-    (fill yes (arc_segments 32) (thermal_gap 0.508) (thermal_bridge_width 0.508))
-    (polygon
-      (pts
-        (xy 198.247 145.161) (xy 186.817 145.161) (xy 186.817 63.373) (xy 143.383 63.373) (xy 143.383 145.161)
-        (xy 134.366 145.161) (xy 134.366 39.624) (xy 198.247 39.624)
-      )
-    )
